File: PCB/UMTK_V1_5/S4_HX711.kicad_sch (KiCad schematic)
At the start: 12 parts, among them Q9 Q_PNP_BEC, U1 HX711

Commit message: Schematic Done, Assigning footprint
Parts:
- gave numbers to parts that had none: 1
- renumbered C11 to C13, C12 to C14, C14 to C15, C13 to C16, Q9 to Q1, R58 to R28, R59 to R29, R56 to R30, R57 to R31, R60 to R32, U1 to U2
Changed lines of the file:
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@@
 		(on_board yes)
 		(dnp no)
-		(property "Reference" "R58"
+		(property "Reference" "R28"
 			(at 91.948 102.87 90)
 			(effects
@@
 			(project "UMTK"
 				(path "/2bf3ea67-58b8-47b3-a768-ea6950b40edf/b421850b-f091-436d-99dc-672cc95b7600"
-					(reference "R58")
+					(reference "R28")
 					(unit 1)
 				)
@@
 		(on_board yes)
 		(dnp no)
-		(property "Reference" "#PWR0138"
+		(property "Reference" "#PWR032"
 			(at 165.1 142.24 0)
 			(effects
@@
 			(project "UMTK"
 				(path "/2bf3ea67-58b8-47b3-a768-ea6950b40edf/b421850b-f091-436d-99dc-672cc95b7600"
-					(reference "#PWR0138")
+					(reference "#PWR032")
 					(unit 1)
 				)
@@
 		(on_board yes)
 		(dnp no)
-		(property "Reference" "R60"
+		(property "Reference" "R32"
 			(at 146.304 92.71 90)
 			(effects
@@
 			(project "UMTK"
 				(path "/2bf3ea67-58b8-47b3-a768-ea6950b40edf/b421850b-f091-436d-99dc-672cc95b7600"
-					(reference "R60")
+					(reference "R32")
 					(unit 1)
 				)
@@
 		(on_board yes)
 		(dnp no)
-		(property "Reference" "R56"
+		(property "Reference" "R30"
 			(at 110.998 116.84 90)
 			(effects
@@
 			(project ""
 				(path "/2bf3ea67-58b8-47b3-a768-ea6950b40edf/b421850b-f091-436d-99dc-672cc95b7600"
-					(reference "R56")
+					(reference "R30")
 					(unit 1)
 				)
@@
 		(on_board yes)
 		(dnp no)
-		(property "Reference" "R57"
+		(property "Reference" "R31"
 			(at 110.998 124.46 90)
 			(effects
@@
 			(project "UMTK"
 				(path "/2bf3ea67-58b8-47b3-a768-ea6950b40edf/b421850b-f091-436d-99dc-672cc95b7600"
-					(reference "R57")
+					(reference "R31")
 					(unit 1)
 				)
@@
 		(dnp no)
 		(fields_autoplaced yes)
-		(property "Reference" "U1"
+		(property "Reference" "U2"
 			(at 167.2941 130.81 0)
 			(effects
@@
 			(project ""
 				(path "/2bf3ea67-58b8-47b3-a768-ea6950b40edf/b421850b-f091-436d-99dc-672cc95b7600"
-					(reference "U1")
+					(reference "U2")
 					(unit 1)
 				)
@@
 		(on_board yes)
 		(dnp no)
-		(property "Reference" "C12"
+		(property "Reference" "C14"
 			(at 116.586 120.904 0)
 			(effects
@@
 			(project "UMTK"
 				(path "/2bf3ea67-58b8-47b3-a768-ea6950b40edf/b421850b-f091-436d-99dc-672cc95b7600"
-					(reference "C12")
+					(reference "C14")
 					(unit 1)
 				)
@@
 		(dnp no)
 		(fields_autoplaced yes)
-		(property "Reference" "Q9"
+		(property "Reference" "Q1"
 			(at 130.81 91.4399 0)
 			(effects
@@
 			(project ""
 				(path "/2bf3ea67-58b8-47b3-a768-ea6950b40edf/b421850b-f091-436d-99dc-672cc95b7600"
-					(reference "Q9")
+					(reference "Q1")
 					(unit 1)
 				)
@@
 		(dnp no)
 		(fields_autoplaced yes)
-		(property "Reference" "C13"
+		(property "Reference" "C16"
 			(at 175.26 80.01 90)
 			(effects
@@
 			(project "UMTK"
 				(path "/2bf3ea67-58b8-47b3-a768-ea6950b40edf/b421850b-f091-436d-99dc-672cc95b7600"
-					(reference "C13")
+					(reference "C16")
 					(unit 1)
 				)
@@
 		(on_board yes)
 		(dnp no)
-		(property "Reference" "C14"
+		(property "Reference" "C15"
 			(at 150.876 133.604 0)
 			(effects
@@
 			(project "UMTK"
 				(path "/2bf3ea67-58b8-47b3-a768-ea6950b40edf/b421850b-f091-436d-99dc-672cc95b7600"
-					(reference "C14")
+					(reference "C15")
 					(unit 1)
 				)
@@
 		(dnp no)
 		(fields_autoplaced yes)
-		(property "Reference" "#PWR041"
+		(property "Reference" "#PWR033"
 			(at 167.64 81.28 0)
 			(effects
@@
 			(project ""
 				(path "/2bf3ea67-58b8-47b3-a768-ea6950b40edf/b421850b-f091-436d-99dc-672cc95b7600"
-					(reference "#PWR041")
+					(reference "#PWR033")
 					(unit 1)
 				)
@@
 		(dnp no)
 		(fields_autoplaced yes)
-		(property "Reference" "#PWR0142"
+		(property "Reference" "#PWR031"
 			(at 153.67 81.28 0)
 			(effects
@@
 			(project "UMTK"
 				(path "/2bf3ea67-58b8-47b3-a768-ea6950b40edf/b421850b-f091-436d-99dc-672cc95b7600"
-					(reference "#PWR0142")
+					(reference "#PWR031")
 					(unit 1)
 				)
@@
 		(on_board yes)
 		(dnp no)
-		(property "Reference" "#PWR0139"
+		(property "Reference" "#PWR034"
 			(at 182.88 87.63 0)
 			(effects
@@
 			(project "UMTK"
 				(path "/2bf3ea67-58b8-47b3-a768-ea6950b40edf/b421850b-f091-436d-99dc-672cc95b7600"
-					(reference "#PWR0139")
+					(reference "#PWR034")
 					(unit 1)
 				)
@@
 		(dnp no)
 		(fields_autoplaced yes)
-		(property "Reference" "C11"
+		(property "Reference" "C13"
 			(at 55.88 100.3299 0)
 			(effects
@@
 			(project "UMTK"
 				(path "/2bf3ea67-58b8-47b3-a768-ea6950b40edf/b421850b-f091-436d-99dc-672cc95b7600"
-					(reference "C11")
+					(reference "C13")
 					(unit 1)
 				)
@@
 		(on_board yes)
 		(dnp no)
-		(property "Reference" "R59"
+		(property "Reference" "R29"
 			(at 86.614 110.998 90)
 			(effects
@@
 			(project "UMTK"
 				(path "/2bf3ea67-58b8-47b3-a768-ea6950b40edf/b421850b-f091-436d-99dc-672cc95b7600"
-					(reference "R59")
+					(reference "R29")
 					(unit 1)
 				)
@@
 		(on_board yes)
 		(dnp no)
-		(property "Reference" "#PWR0137"
+		(property "Reference" "#PWR030"
 			(at 74.93 109.22 0)
 			(effects
@@
 			(project "UMTK"
 				(path "/2bf3ea67-58b8-47b3-a768-ea6950b40edf/b421850b-f091-436d-99dc-672cc95b7600"
-					(reference "#PWR0137")
+					(reference "#PWR030")
 					(unit 1)
 				)
@@
 		(on_board yes)
 		(dnp no)
-		(property "Reference" "J?"
+		(property "Reference" "J3"
 			(at 64.516 65.786 0)
 			(effects
@@
 			(project ""
 				(path "/2bf3ea67-58b8-47b3-a768-ea6950b40edf/b421850b-f091-436d-99dc-672cc95b7600"
-					(reference "J?")
+					(reference "J3")
 					(unit 1)
 				)
@@
 		(on_board yes)
 		(dnp no)
-		(property "Reference" "#PWR0141"
+		(property "Reference" "#PWR035"
 			(at 198.12 113.03 0)
 			(effects
@@
 			(project "UMTK"
 				(path "/2bf3ea67-58b8-47b3-a768-ea6950b40edf/b421850b-f091-436d-99dc-672cc95b7600"
-					(reference "#PWR0141")
-					(unit 1)
-				)
+					(reference "#PWR035")
+					(unit 1)
+				)

Commit message: Footprint assign
Parts:
- C13, C16: footprint (none) -> Diode_SMD:D_1206_3216Metric
- C14, C15: footprint (none) -> Capacitor_SMD:C_0402_1005Metric
- J3: footprint 4Pin JST -> Connector_JST:JST_XH_B4B-XH-A_1x04_P2.50mm_Vertical
- Q1: footprint (none) -> Package_TO_SOT_SMD:SOT-23
- R28, R29, R30, R31, R32: footprint (none) -> Resistor_SMD:R_0402_1005Metric
Changed lines of the file:
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@@
 			)
 		)
-		(property "Footprint" ""
+		(property "Footprint" "Resistor_SMD:R_0402_1005Metric"
 			(at 91.694 104.394 90)
 			(effects
@@
 			)
 		)
-		(property "Footprint" ""
+		(property "Footprint" "Resistor_SMD:R_0402_1005Metric"
 			(at 146.304 94.234 90)
 			(effects
@@
 			)
 		)
-		(property "Footprint" ""
+		(property "Footprint" "Resistor_SMD:R_0402_1005Metric"
 			(at 109.474 118.364 90)
 			(effects
@@
 			)
 		)
-		(property "Footprint" ""
+		(property "Footprint" "Resistor_SMD:R_0402_1005Metric"
 			(at 109.474 125.984 90)
 			(effects
@@
 			)
 		)
-		(property "Footprint" ""
+		(property "Footprint" "Capacitor_SMD:C_0402_1005Metric"
 			(at 116.5352 127 0)
 			(effects
@@
 			)
 		)
-		(property "Footprint" ""
+		(property "Footprint" "Package_TO_SOT_SMD:SOT-23"
 			(at 130.81 95.25 0)
 			(effects
@@
 			)
 		)
-		(property "Footprint" ""
+		(property "Footprint" "Diode_SMD:D_1206_3216Metric"
 			(at 179.07 86.6648 0)
 			(effects
@@
 			)
 		)
-		(property "Footprint" ""
+		(property "Footprint" "Capacitor_SMD:C_0402_1005Metric"
 			(at 150.8252 139.7 0)
 			(effects
@@
 			)
 		)
-		(property "Footprint" ""
+		(property "Footprint" "Diode_SMD:D_1206_3216Metric"
 			(at 51.1048 97.79 0)
 			(effects
@@
 			)
 		)
-		(property "Footprint" ""
+		(property "Footprint" "Resistor_SMD:R_0402_1005Metric"
 			(at 91.694 112.014 90)
 			(effects
@@
 			)
 		)
-		(property "Footprint" "4Pin JST"
+		(property "Footprint" "Connector_JST:JST_XH_B4B-XH-A_1x04_P2.50mm_Vertical"
 			(at 69.85 78.74 0)
 			(effects

Commit message: Initial Place, Board Stack
Parts:
- C13, C16: footprint Diode_SMD:D_1206_3216Metric -> Capacitor_SMD:C_0805_2012Metric
Changed lines of the file:
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@@
 			)
 		)
-		(property "Footprint" "Diode_SMD:D_1206_3216Metric"
+		(property "Footprint" "Capacitor_SMD:C_0805_2012Metric"
 			(at 179.07 86.6648 0)
 			(effects
@@
 			)
 		)
-		(property "Footprint" "Diode_SMD:D_1206_3216Metric"
+		(property "Footprint" "Capacitor_SMD:C_0805_2012Metric"
 			(at 51.1048 97.79 0)
 			(effects

Commit message: Routing
Parts:
- J3: value JST 4pin -> LOADCELL; footprint Connector_JST:JST_XH_B4B-XH-A_1x04_P2.50mm_Vertical -> Connector_Phoenix_MC:PhoenixContact_MC_1,5_4-G-3.81_1x04_P3.81mm_Horizontal
Connections:
- net LCS+: now also J3.2; no longer J3.3
- net LCS-: now also J3.3; no longer J3.2
Changed lines of the file:
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@@
 	(wire
 		(pts
-			(xy 74.93 71.12) (xy 82.55 71.12)
+			(xy 99.06 104.14) (xy 99.06 105.41)
+		)
+		(stroke
+			(width 0)
+			(type default)
+		)
+	)
+	(wire
+		(pts
+			(xy 146.05 113.03) (xy 152.4 113.03)
+		)
+		(stroke
+			(width 0)
+			(type default)
+		)
+	)
+	(wire
+		(pts
+			(xy 115.57 127) (xy 146.05 127)
+		)
+		(stroke
+			(width 0)
+			(type default)
+		)
+	)
+	(wire
+		(pts
+			(xy 149.86 139.7) (xy 165.1 139.7)
+		)
+		(stroke
+			(width 0)
+			(type default)
+		)
+	)
+	(wire
+		(pts
+			(xy 113.03 127) (xy 115.57 127)
+		)
+		(stroke
+			(width 0)
+			(type default)
+		)
+	)
+	(wire
+		(pts
+			(xy 74.93 73.66) (xy 82.55 73.66)
 		)
 		(stroke
@@
 	(wire
 		(pts
-			(xy 99.06 104.14) (xy 99.06 105.41)
-		)
-		(stroke
-			(width 0)
-			(type default)
-		)
-	)
-	(wire
-		(pts
-			(xy 146.05 113.03) (xy 152.4 113.03)
-		)
-		(stroke
-			(width 0)
-			(type default)
-		)
-	)
-	(wire
-		(pts
-			(xy 115.57 127) (xy 146.05 127)
-		)
-		(stroke
-			(width 0)
-			(type default)
-		)
-	)
-	(wire
-		(pts
-			(xy 149.86 139.7) (xy 165.1 139.7)
-		)
-		(stroke
-			(width 0)
-			(type default)
-		)
-	)
-	(wire
-		(pts
-			(xy 113.03 127) (xy 115.57 127)
-		)
-		(stroke
-			(width 0)
-			(type default)
-		)
-	)
-	(wire
-		(pts
 			(xy 146.05 127) (xy 146.05 113.03)
 		)
@@
 	(wire
 		(pts
+			(xy 82.55 71.12) (xy 74.93 71.12)
+		)
+		(stroke
+			(width 0.254)
+			(type default)
+		)
+	)
+	(wire
+		(pts
 			(xy 167.64 87.63) (xy 171.45 87.63)
 		)
@@
 		(stroke
 			(width 0)
-			(type default)
-		)
-	)
-	(wire
-		(pts
-			(xy 82.55 73.66) (xy 74.93 73.66)
-		)
-		(stroke
-			(width 0.254)
 			(type default)
 		)
@@
 		)
 	)
-	(label "LCS+"
-		(at 82.55 71.12 0)
+	(label "LCS-"
+		(at 40.64 127 180)
 		(fields_autoplaced yes)
 		(effects
@@
 				(size 1.27 1.27)
 			)
-			(justify left bottom)
-		)
-	)
-	(label "LCS-"
-		(at 40.64 127 180)
+			(justify right bottom)
+		)
+	)
+	(label "LCE+"
+		(at 82.55 68.58 0)
 		(fields_autoplaced yes)
 		(effects
@@
 				(size 1.27 1.27)
 			)
-			(justify right bottom)
+			(justify left bottom)
 		)
 	)
 	(label "LCS-"
-		(at 82.55 73.66 0)
+		(at 82.55 71.12 0)
 		(fields_autoplaced yes)
 		(effects
@@
 		)
 	)
-	(label "LCE+"
-		(at 82.55 68.58 0)
+	(label "LCS+"
+		(at 82.55 73.66 0)
 		(fields_autoplaced yes)
 		(effects
@@
 			)
 		)
-		(property "Value" "JST 4pin"
+		(property "Value" "LOADCELL"
 			(at 64.516 81.534 0)
 			(effects
@@
 			)
 		)
-		(property "Footprint" "Connector_JST:JST_XH_B4B-XH-A_1x04_P2.50mm_Vertical"
+		(property "Footprint" "Connector_Phoenix_MC:PhoenixContact_MC_1,5_4-G-3.81_1x04_P3.81mm_Horizontal"
 			(at 69.85 78.74 0)
 			(effects

Commit message: Routing and JLC Assignment Done
Parts:
- R28: footprint Resistor_SMD:R_0402_1005Metric -> Capacitor_SMD:C_0603_1608Metric
Changed lines of the file:
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@@
 			)
 		)
-		(property "Footprint" "Resistor_SMD:R_0402_1005Metric"
+		(property "Footprint" "Capacitor_SMD:C_0603_1608Metric"
 			(at 91.694 104.394 90)
 			(effects

Commit message: Make simple components bigger
Parts:
- C14, C15: footprint Capacitor_SMD:C_0402_1005Metric -> Capacitor_SMD:C_0603_1608Metric
- R29, R30, R31, R32: footprint Resistor_SMD:R_0402_1005Metric -> Resistor_SMD:R_0603_1608Metric
Changed lines of the file:
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@@
 			)
 		)
-		(property "Footprint" "Resistor_SMD:R_0402_1005Metric"
+		(property "Footprint" "Resistor_SMD:R_0603_1608Metric"
 			(at 146.304 94.234 90)
 			(effects
@@
 			)
 		)
-		(property "Footprint" "Resistor_SMD:R_0402_1005Metric"
+		(property "Footprint" "Resistor_SMD:R_0603_1608Metric"
 			(at 109.474 118.364 90)
 			(effects
@@
 			)
 		)
-		(property "Footprint" "Resistor_SMD:R_0402_1005Metric"
+		(property "Footprint" "Resistor_SMD:R_0603_1608Metric"
 			(at 109.474 125.984 90)
 			(effects
@@
 			)
 		)
-		(property "Footprint" "Capacitor_SMD:C_0402_1005Metric"
+		(property "Footprint" "Capacitor_SMD:C_0603_1608Metric"
 			(at 116.5352 127 0)
 			(effects
@@
 			)
 		)
-		(property "Footprint" "Capacitor_SMD:C_0402_1005Metric"
+		(property "Footprint" "Capacitor_SMD:C_0603_1608Metric"
 			(at 150.8252 139.7 0)
 			(effects
@@
 			)
 		)
-		(property "Footprint" "Resistor_SMD:R_0402_1005Metric"
+		(property "Footprint" "Resistor_SMD:R_0603_1608Metric"
 			(at 91.694 112.014 90)
 			(effects
