File: PCB/_autosave-UMTK.kicad_pcb (KiCad board)
At the start: 4 copper layers, 170 x 80 mm, 121 parts, among them J1 Motor Out, J2 ESTOP, J3 LOADCELL, J5 PJ-102BH, J8 10033526-N3212LF, Q1 Q_PNP_BEC, U1 DRV8873SPWPRQ1, U10 LM2576HVS-5, U11 SN74LVC1T45DCK, U12 SN74LVC1T45DCK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

Commit message: Schematic bit done for adding arduino, improved motor maybe a bit by adding caps, improved slide a bit by adding protection and more caps
Parts:
- moved C27 233.6 mm to (-35.0, 88.9)
- moved C28 233.6 mm to (-35.0, 91.4)
- moved C29 233.6 mm to (-35.0, 93.9)
- moved C30 233.6 mm to (-35.0, 96.4)
- moved C31 233.6 mm to (-35.0, 98.9)
- moved R10 233.6 mm to (-63.4, 73.4)
- moved R11 233.6 mm to (-63.4, 75.9)
- moved R12 233.6 mm to (-63.4, 78.4)
- moved R13 233.6 mm to (-63.4, 80.9)
- moved R14 233.6 mm to (-63.4, 83.4)
- moved R15 233.6 mm to (-63.4, 85.9)
- moved U5 233.6 mm to (-40.0, 92.9)
- moved U9 233.6 mm to (-52.8, 104.6)
- moved C32 233.6 mm to (-53.1, 108.3)
- moved C33 233.6 mm to (-45.4, 103.9)
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