File: PCB/UMTK.kicad_pcb (KiCad board)
At the start: 4 copper layers, 170 x 80 mm, 121 parts, among them J1 Motor Out, J2 ESTOP, J3 LOADCELL, J5 PJ-102BH, J8 10033526-N3212LF, Q1 Q_PNP_BEC, U1 DRV8873SPWPRQ1, U10 LM2576HVS-5, U11 SN74LVC1T45DCK, U12 SN74LVC1T45DCK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

Commit message: Changed power stage, there as a mistake, also generally changing lots of stuff
Parts:
- removed C17: 100u hv, Capacitor_SMD:CP_Elec_10x10.5
- removed C21: 1000u, Capacitor_SMD:CP_Elec_8x10.5
- removed D1: MBR0560, Diode_SMD:D_SOD-123
- removed L1: 100u, Inductor_SMD:L_Sunlord_MWSA1206S-101
- removed U10: LM2576HVS-5, Package_TO_SOT_SMD:TO-263-5_TabPin3
- added C25: 33p, Capacitor_SMD:C_0603_1608Metric, F.Cu at (-58.0, 50.1)
- added C26: 33p, Capacitor_SMD:C_0603_1608Metric, F.Cu at (-58.0, 52.6)
- added C34: 33p, Capacitor_SMD:C_0603_1608Metric, F.Cu at (-58.0, 55.1)
- added C35: 33p, Capacitor_SMD:C_0603_1608Metric, F.Cu at (-58.0, 57.6)
- added C40: 10u HV, Capacitor_SMD:CP_Elec_6.3x5.4, F.Cu at (203.2, 64.0)
- added C41: 1u hv, Capacitor_SMD:C_0603_1608Metric, F.Cu at (-42.3, 37.6)
- added C42: 220n, Capacitor_SMD:C_0603_1608Metric, F.Cu at (-42.3, 40.1)
- added C43: 0u1, Capacitor_SMD:C_0603_1608Metric, F.Cu at (-42.3, 42.6)
- added C44: 22u, Capacitor_SMD:C_1210_3225Metric, F.Cu at (-47.1, 38.5)
- added C45: 22u, Capacitor_SMD:C_1210_3225Metric, F.Cu at (-47.1, 42.7)
- added C46: 22u, Capacitor_SMD:C_1210_3225Metric, F.Cu at (-47.1, 47.0)
- added C47: 22u, Capacitor_SMD:C_1210_3225Metric, F.Cu at (-47.1, 51.2)
- added C48: DNP, Capacitor_SMD:C_1206_3216Metric, F.Cu at (-47.1, 55.0)
- added D5: SS34, Diode_SMD:D_SMA, F.Cu at (-67.6, 61.6)
- added D6: SS34, Diode_SMD:D_SMA, F.Cu at (-45.9, 62.2)
- added F2: Polyfuse, Fuse:Fuse_0805_2012Metric, F.Cu at (-54.8, 37.8)
- added J4: USB_C_Receptacle_USB2.0_16P, Connector_USB:USB_C_Receptacle_HRO_TYPE-C-31-M-12, F.Cu at (47.9, 23.4)
- added L2: 10uH, Inductor_SMD:L_Changjiang_FXL0530, F.Cu at (-36.5, 54.6)
- added R40: 5K1, Resistor_SMD:R_0603_1608Metric, F.Cu at (-58.0, 60.1)
- added R41: 100K, Resistor_SMD:R_0603_1608Metric, F.Cu at (-42.3, 45.1)
- added R42: 1K, Resistor_SMD:R_0603_1608Metric, F.Cu at (-58.0, 62.6)
- added R43: 100K, Resistor_SMD:R_0603_1608Metric, F.Cu at (-42.3, 47.6)
- added R44: 100r, Resistor_SMD:R_0603_1608Metric, F.Cu at (-54.0, 50.1)
- added R45: 100r, Resistor_SMD:R_0603_1608Metric, F.Cu at (-54.0, 52.6)
- added R46: 2K, Resistor_SMD:R_0603_1608Metric, F.Cu at (-54.0, 55.1)
- added R47: 2K, Resistor_SMD:R_0603_1608Metric, F.Cu at (-54.0, 57.6)
- added R48: 5K1, Resistor_SMD:R_0603_1608Metric, F.Cu at (-54.0, 60.1)
- added R49: 24K9, Resistor_SMD:R_0603_1608Metric, F.Cu at (-42.3, 50.1)
- added U14: LMR33620ADDA, Package_SO:Texas_HSOP-8-1EP_3.9x4.9mm_P1.27mm_ThermalVias, F.Cu at (-25.3, 25.3)
- added Y1: HC49 16Mhz, Crystal:Crystal_SMD_HC49-SD, F.Cu at (-67.6, 37.1)
- added Y2: HC49-12M, Crystal:Crystal_SMD_HC49-SD, F.Cu at (-50.0, 20.8)
- moved C27 233.6 mm to (-35.0, 88.9)
- moved C28 233.6 mm to (-35.0, 91.4)
- moved C29 233.6 mm to (-35.0, 93.9)
- moved C30 233.6 mm to (-35.0, 96.4)
- moved C31 233.6 mm to (-35.0, 98.9)
- moved R10 233.6 mm to (-63.4, 73.4)
- moved R11 233.6 mm to (-63.4, 75.9)
- moved R12 233.6 mm to (-63.4, 78.4)
- moved R13 233.6 mm to (-63.4, 80.9)
- moved R14 233.6 mm to (-63.4, 83.4)
- moved R15 233.6 mm to (-63.4, 85.9)
- moved U9 233.6 mm to (-52.8, 104.6)
- moved C32 233.6 mm to (-53.1, 108.3)
- moved C33 233.6 mm to (-45.4, 103.9)
- moved C36 233.6 mm to (-31.0, 88.9)
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Connections:
- net Net-(U4-~{DTR}) renamed /Arduino/DTR
- C28 pad 2: /Arduino/ARDUINO_VCC -> +5V
- C29 pad 2: /Arduino/ARDUINO_VCC -> +5V
- C30 pad 2: /Arduino/ARDUINO_VCC -> +5V
- R7 pad 1: +3V3 -> Net-(D6-K)
- U3 pad 10: /Arduino/ARDUINO_VCC -> +5V
- U3 pad 100: /Arduino/ARDUINO_VCC -> +5V
- U3 pad 31: /Arduino/ARDUINO_VCC -> +5V
- U3 pad 61: /Arduino/ARDUINO_VCC -> +5V
- U3 pad 80: /Arduino/ARDUINO_VCC -> +5V
Routing:
- net GNDA: track 96.9 -> 78.0 mm, vias 386 -> 364
- net +5V: track 119.1 -> 112.5 mm, vias 61 -> 43
- net Net-(D1-K): track 4.12 -> 0.00 mm
- removed copper zone on F.Cu, net Net-(D1-K)

Commit message: Progress save, schematic done
Parts:
- removed R7: 0R, Resistor_SMD:R_0603_1608Metric
- moved C5 241.6 mm to (174.2, 81.0), turned to -90 degrees
- moved R18 234.2 mm to (174.5, 90.0), turned to 90 degrees
- moved R17 234.1 mm to (174.5, 85.6), turned to 90 degrees
- moved C4 228.4 mm to (161.0, 81.0), turned to -90 degrees
- moved R15 224.4 mm to (161.0, 85.3), turned to 90 degrees
- moved R16 221.0 mm to (161.0, 89.9), turned to 90 degrees
- moved C3 215.2 mm to (147.8, 80.8), turned to -90 degrees
- moved R14 211.3 mm to (147.8, 89.7), turned to 90 degrees
- moved R13 211.3 mm to (147.8, 85.7), turned to 90 degrees
- moved C2 202.3 mm to (134.9, 81.3), turned to -90 degrees
- moved R12 198.6 mm to (134.9, 89.9), turned to 90 degrees
- moved R11 198.5 mm to (134.9, 85.6), turned to 90 degrees
- moved C1 189.0 mm to (121.4, 82.0), turned to -90 degrees
- moved R9 188.8 mm to (121.4, 85.7), turned to 90 degrees
- moved U9 186.5 mm to (119.6, 33.5), turned to 180 degrees
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Connections:
- C24 pad 1: Net-(J8-ID) -> Net-(D6-K)
- C32 pad 1: Net-(J8-ID) -> Net-(D6-K)
- J8 pad 4: Net-(J8-ID) -> Net-(D6-K)
- U9 pad 1: Net-(R2-Pad2) -> Net-(R3-Pad2)
- U9 pad 3: Net-(R3-Pad2) -> Net-(R2-Pad2)
- U9 pad 4: Net-(J8-D-) -> Net-(J8-VBUS)
- U9 pad 6: Net-(J8-VBUS) -> Net-(J8-D-)
Routing:
- net (no net): track 538.0 -> 0.00 mm, vias 13 -> 0
- net /Arduino/A12: track 0.00 -> 126.8 mm, vias 0 -> 3
- net /Arduino/A11: track 0.00 -> 114.7 mm, vias 0 -> 4
- net /Arduino/A10: track 0.00 -> 106.0 mm, vias 0 -> 3
- net /Arduino/A9: track 0.00 -> 90.7 mm, vias 0 -> 3
- net /Arduino/A1: track 93.8 -> 8.01 mm
- net /Arduino/A8: track 0.00 -> 71.3 mm, vias 0 -> 1
- net Net-(R3-Pad2): track 0.00 -> 69.6 mm, vias 0 -> 1
- net Net-(R2-Pad2): track 0.00 -> 68.2 mm, vias 0 -> 1
- net /Arduino/D3: track 48.3 -> 0.00 mm
- net /Arduino/D23: track 42.0 -> 0.00 mm, vias 1 -> 0
- net Net-(J8-ID): track 26.6 -> 0.00 mm
- net Net-(J8-D+): track 38.6 -> 15.6 mm
- net Net-(D6-K): track 0.00 -> 20.9 mm
- net /Linear Slide/_SLIDE_DAT_: track 16.9 -> 0.00 mm, vias 2 -> 0
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
Commit message: Update
Parts:
- removed C40: 10u HV, Capacitor_SMD:CP_Elec_6.3x5.4
- moved C41 29.7 mm to (-13.2, 43.7)
- moved R43 29.2 mm to (-13.2, 45.5), turned to 180 degrees
- moved C43 28.4 mm to (-14.0, 41.1), turned to -90 degrees
- moved R49 25.7 mm to (-16.8, 47.2)
- moved L2 24.9 mm to (-19.3, 36.6), turned to 180 degrees
- moved R41 20.4 mm to (-23.1, 52.1), turned to 180 degrees
- moved U14 19.0 mm to (-19.5, 43.3)
- moved C42 17.7 mm to (-24.6, 41.7), turned to 90 degrees
- moved C37 14.6 mm to (-29.3, 105.9)
- moved R56 14.6 mm to (-29.3, 113.4)
- moved C28 14.6 mm to (-33.3, 105.9)
- moved C31 14.6 mm to (-33.3, 113.4)
- moved D14 14.6 mm to (-33.2, 90.5)
- moved D17 14.6 mm to (-33.2, 93.1)
- moved D20 14.6 mm to (-33.2, 100.8)
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Routing:
- net +3V3: track 41.2 -> 46.0 mm
- net Net-(C5-Pad2): track 12.5 -> 14.4 mm
- net +5V: track 112.7 -> 113.0 mm, vias 40 -> 39
- net GNDA: vias 359 -> 316
- net /Arduino/A11: vias 4 -> 3

Commit message: Laying out
Parts:
- added C50: 10u HV, Capacitor_SMD:C_1210_3225Metric, F.Cu at (155.2, 63.1)
- C48: footprint Capacitor_SMD:C_1206_3216Metric -> Capacitor_SMD:C_0603_1608Metric
- F2: footprint Fuse:Fuse_0805_2012Metric -> Fuse:Fuse_1206_3216Metric
- J4: footprint Connector_USB:USB_C_Receptacle_HRO_TYPE-C-31-M-12 -> Connector_USB:USB_C_Receptacle_HCTL_HC-TYPE-C-16P-01A
- L2: footprint Inductor_SMD:L_Changjiang_FXL0530 -> Inductor_SMD:L_Changjiang_FXL0630
- moved C46 210.5 mm to (162.3, 67.9), turned to 90 degrees
- moved C45 207.4 mm to (158.8, 67.9), turned to 90 degrees
- moved C44 204.4 mm to (155.2, 67.9), turned to 90 degrees
- moved C47 203.4 mm to (155.2, 72.7), turned to -90 degrees
- moved C48 188.7 mm to (141.6, 58.4), turned to 180 degrees
- moved C42 178.3 mm to (152.2, 63.8), turned to -90 degrees
- moved R41 174.4 mm to (151.2, 57.8), turned to 90 degrees
- moved L2 169.9 mm to (147.3, 70.0), turned to 0 degrees
- moved U14 167.9 mm to (147.3, 62.8), turned to 180 degrees
- moved R49 162.3 mm to (145.1, 58.8), turned to 180 degrees
- moved C43 157.7 mm to (142.0, 64.5), turned to 90 degrees
- moved C41 155.9 mm to (141.6, 62.0), turned to 180 degrees
- moved R43 155.5 mm to (141.6, 60.2)
- moved R46 114.1 mm to (56.6, 26.9), turned to 90 degrees
- moved R47 111.7 mm to (53.5, 26.9), turned to 90 degrees
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Routing:
- net /Power/LMR_VCC: track 0.00 -> 21.3 mm, vias 0 -> 2
- net Net-(D14-K): track 0.00 -> 15.5 mm, vias 0 -> 2
- net Net-(D13-K): track 0.00 -> 15.5 mm
- net Net-(U4-XI): track 0.00 -> 14.6 mm
- net Net-(U4-XO): track 0.00 -> 13.6 mm
- net GNDA: track 68.7 -> 75.2 mm, vias 316 -> 319
- net Net-(U14-FB): track 0.00 -> 6.44 mm
- net /Arduino/A3: track 87.0 -> 81.4 mm
- net Net-(U14-BOOT): track 0.00 -> 2.79 mm
- net /Power/PG: track 0.00 -> 2.72 mm
- net +12V: track 9.05 -> 11.6 mm, vias 50 -> 48
- net Net-(D14-A): track 0.00 -> 2.58 mm
- net Net-(D13-A): track 0.00 -> 2.58 mm
- net +5V: track 113.0 -> 114.8 mm, vias 39 -> 58
- added copper zone on F.Cu, net Net-(U14-SW)
